Commit message: Add moveit_resources_ prefix to pr2_description

File: pr2_description/robots/pr2.urdf.xacro (robot description, xacro)
@@ -3,29 +3,29 @@
   <!-- The following included files set up definitions of parts of the robot body -->
   <!-- misc common stuff? -->
-  <xacro:include filename="$(find pr2_description)/urdf/common.xacro" />
+  <xacro:include filename="$(find moveit_resources_pr2_description)/urdf/common.xacro" />
   <!-- PR2 Arm -->
-  <xacro:include filename="$(find pr2_description)/urdf/shoulder_v0/shoulder.urdf.xacro" />
-  <xacro:include filename="$(find pr2_description)/urdf/upper_arm_v0/upper_arm.urdf.xacro" />
-  <xacro:include filename="$(find pr2_description)/urdf/forearm_v0/forearm.urdf.xacro" />
+  <xacro:include filename="$(find moveit_resources_pr2_description)/urdf/shoulder_v0/shoulder.urdf.xacro" />
+  <xacro:include filename="$(find moveit_resources_pr2_description)/urdf/upper_arm_v0/upper_arm.urdf.xacro" />
+  <xacro:include filename="$(find moveit_resources_pr2_description)/urdf/forearm_v0/forearm.urdf.xacro" />
   <!-- PR2 gripper -->
-  <xacro:include filename="$(find pr2_description)/urdf/gripper_v0/gripper.urdf.xacro" />
+  <xacro:include filename="$(find moveit_resources_pr2_description)/urdf/gripper_v0/gripper.urdf.xacro" />
   <!-- PR2 head -->
-  <xacro:include filename="$(find pr2_description)/urdf/head_v0/head.urdf.xacro" />
+  <xacro:include filename="$(find moveit_resources_pr2_description)/urdf/head_v0/head.urdf.xacro" />
   <!-- PR2 tilting laser mount -->
-  <xacro:include filename="$(find pr2_description)/urdf/tilting_laser_v0/tilting_laser.urdf.xacro" />
+  <xacro:include filename="$(find moveit_resources_pr2_description)/urdf/tilting_laser_v0/tilting_laser.urdf.xacro" />
   <!-- PR2 torso -->
-  <xacro:include filename="$(find pr2_description)/urdf/torso_v0/torso.urdf.xacro" />
+  <xacro:include filename="$(find moveit_resources_pr2_description)/urdf/torso_v0/torso.urdf.xacro" />
   <!-- PR2 base -->
-  <xacro:include filename="$(find pr2_description)/urdf/base_v0/base.urdf.xacro" />
+  <xacro:include filename="$(find moveit_resources_pr2_description)/urdf/base_v0/base.urdf.xacro" />
   <!-- Head sensors -->
-  <xacro:include filename="$(find pr2_description)/urdf/sensors/head_sensor_package.urdf.xacro" />
+  <xacro:include filename="$(find moveit_resources_pr2_description)/urdf/sensors/head_sensor_package.urdf.xacro" />
   <!-- Camera sensors -->
-  <xacro:include filename="$(find pr2_description)/urdf/sensors/wge100_camera.urdf.xacro" />
+  <xacro:include filename="$(find moveit_resources_pr2_description)/urdf/sensors/wge100_camera.urdf.xacro" />
   <!-- Texture projector -->
-  <xacro:include filename="$(find pr2_description)/urdf/sensors/projector_wg6802418.urdf.xacro" />
+  <xacro:include filename="$(find moveit_resources_pr2_description)/urdf/sensors/projector_wg6802418.urdf.xacro" />
   <!-- generic simulator_gazebo plugins for starting mechanism control, ros time, ros battery -->
-  <xacro:include filename="$(find pr2_description)/gazebo/gazebo.urdf.xacro" />
+  <xacro:include filename="$(find moveit_resources_pr2_description)/gazebo/gazebo.urdf.xacro" />
   <!-- materials for visualization -->
-  <xacro:include filename="$(find pr2_description)/urdf/materials.urdf.xacro" />
+  <xacro:include filename="$(find moveit_resources_pr2_description)/urdf/materials.urdf.xacro" />
   <!-- Now we can start using the macros included above to define the actual PR2 -->
   <!-- The first use of a macro.  This one was defined in base.urdf.xacro above.
@@ -123,5 +123,5 @@
   <!-- Kinect2 xacro -->
   <xacro:if value="$(arg KINECT2)">
-    <xacro:include filename="$(find pr2_description)/urdf/sensors/kinect2.urdf.xacro" />
+    <xacro:include filename="$(find moveit_resources_pr2_description)/urdf/sensors/kinect2.urdf.xacro" />
     <xacro:kinect2_v0 name="head_mount" parent="head_plate_frame" >
       <origin xyz="-0.137376 0 0.091746" rpy="0 0 0" />
@@ -131,5 +131,5 @@
   <xacro:unless value="$(arg KINECT2)">
     <xacro:if value="$(arg KINECT1)">
-      <xacro:include filename="$(find pr2_description)/urdf/sensors/kinect_prosilica_camera.urdf.xacro" />
+      <xacro:include filename="$(find moveit_resources_pr2_description)/urdf/sensors/kinect_prosilica_camera.urdf.xacro" />
       <!-- Base of Kinect/Prosilica Mount -->
       <xacro:kinect_prosilica_camera_swept_back_v0 name="head_mount" parent="head_plate_frame" >

File: pr2_description/robots/pr2_no_arms.urdf.xacro (robot description, xacro)
@@ -3,23 +3,23 @@
   <!-- The following included files set up definitions of parts of the robot body -->
   <!-- misc common stuff? -->
-  <xacro:include filename="$(find pr2_description)/urdf/common.xacro" />
+  <xacro:include filename="$(find moveit_resources_pr2_description)/urdf/common.xacro" />
   <!-- PR2 head -->
-  <xacro:include filename="$(find pr2_description)/urdf/head_v0/head.urdf.xacro" />
+  <xacro:include filename="$(find moveit_resources_pr2_description)/urdf/head_v0/head.urdf.xacro" />
   <!-- PR2 tilting laser mount -->
-  <xacro:include filename="$(find pr2_description)/urdf/tilting_laser_v0/tilting_laser.urdf.xacro" />
+  <xacro:include filename="$(find moveit_resources_pr2_description)/urdf/tilting_laser_v0/tilting_laser.urdf.xacro" />
   <!-- PR2 torso -->
-  <xacro:include filename="$(find pr2_description)/urdf/torso_v0/torso.urdf.xacro" />
+  <xacro:include filename="$(find moveit_resources_pr2_description)/urdf/torso_v0/torso.urdf.xacro" />
   <!-- PR2 base -->
-  <xacro:include filename="$(find pr2_description)/urdf/base_v0/base.urdf.xacro" />
+  <xacro:include filename="$(find moveit_resources_pr2_description)/urdf/base_v0/base.urdf.xacro" />
   <!-- Head sensors -->
-  <xacro:include filename="$(find pr2_description)/urdf/sensors/head_sensor_package.urdf.xacro" />
+  <xacro:include filename="$(find moveit_resources_pr2_description)/urdf/sensors/head_sensor_package.urdf.xacro" />
   <!-- Camera sensors -->
-  <xacro:include filename="$(find pr2_description)/urdf/sensors/wge100_camera.urdf.xacro" />
+  <xacro:include filename="$(find moveit_resources_pr2_description)/urdf/sensors/wge100_camera.urdf.xacro" />
   <!-- Texture projector -->
-  <xacro:include filename="$(find pr2_description)/urdf/sensors/projector_wg6802418.urdf.xacro" />
+  <xacro:include filename="$(find moveit_resources_pr2_description)/urdf/sensors/projector_wg6802418.urdf.xacro" />
   <!-- generic simulator_gazebo plugins for starting mechanism control, ros time, ros battery -->
-  <xacro:include filename="$(find pr2_description)/gazebo/gazebo.urdf.xacro" />
+  <xacro:include filename="$(find moveit_resources_pr2_description)/gazebo/gazebo.urdf.xacro" />
   <!-- materials for visualization -->
-  <xacro:include filename="$(find pr2_description)/urdf/materials.urdf.xacro" />
+  <xacro:include filename="$(find moveit_resources_pr2_description)/urdf/materials.urdf.xacro" />
   <!-- Now we can start using the macros included above to define the actual PR2 -->
   <!-- The first use of a macro.  This one was defined in base.urdf.xacro above.

File: pr2_description/robots/pr2_no_kinect.urdf.xacro (robot description, xacro)
@@ -3,29 +3,29 @@
   <!-- The following included files set up definitions of parts of the robot body -->
   <!-- misc common stuff? -->
-  <xacro:include filename="$(find pr2_description)/urdf/common.xacro" />
+  <xacro:include filename="$(find moveit_resources_pr2_description)/urdf/common.xacro" />
   <!-- PR2 Arm -->
-  <xacro:include filename="$(find pr2_description)/urdf/shoulder_v0/shoulder.urdf.xacro" />
-  <xacro:include filename="$(find pr2_description)/urdf/upper_arm_v0/upper_arm.urdf.xacro" />
-  <xacro:include filename="$(find pr2_description)/urdf/forearm_v0/forearm.urdf.xacro" />
+  <xacro:include filename="$(find moveit_resources_pr2_description)/urdf/shoulder_v0/shoulder.urdf.xacro" />
+  <xacro:include filename="$(find moveit_resources_pr2_description)/urdf/upper_arm_v0/upper_arm.urdf.xacro" />
+  <xacro:include filename="$(find moveit_resources_pr2_description)/urdf/forearm_v0/forearm.urdf.xacro" />
   <!-- PR2 gripper -->
-  <xacro:include filename="$(find pr2_description)/urdf/gripper_v0/gripper.urdf.xacro" />
+  <xacro:include filename="$(find moveit_resources_pr2_description)/urdf/gripper_v0/gripper.urdf.xacro" />
   <!-- PR2 head -->
-  <xacro:include filename="$(find pr2_description)/urdf/head_v0/head.urdf.xacro" />
+  <xacro:include filename="$(find moveit_resources_pr2_description)/urdf/head_v0/head.urdf.xacro" />
   <!-- PR2 tilting laser mount -->
-  <xacro:include filename="$(find pr2_description)/urdf/tilting_laser_v0/tilting_laser.urdf.xacro" />
+  <xacro:include filename="$(find moveit_resources_pr2_description)/urdf/tilting_laser_v0/tilting_laser.urdf.xacro" />
   <!-- PR2 torso -->
-  <xacro:include filename="$(find pr2_description)/urdf/torso_v0/torso.urdf.xacro" />
+  <xacro:include filename="$(find moveit_resources_pr2_description)/urdf/torso_v0/torso.urdf.xacro" />
   <!-- PR2 base -->
-  <xacro:include filename="$(find pr2_description)/urdf/base_v0/base.urdf.xacro" />
+  <xacro:include filename="$(find moveit_resources_pr2_description)/urdf/base_v0/base.urdf.xacro" />
   <!-- Head sensors -->
-  <xacro:include filename="$(find pr2_description)/urdf/sensors/head_sensor_package.urdf.xacro" />
+  <xacro:include filename="$(find moveit_resources_pr2_description)/urdf/sensors/head_sensor_package.urdf.xacro" />
   <!-- Camera sensors -->
-  <xacro:include filename="$(find pr2_description)/urdf/sensors/wge100_camera.urdf.xacro" />
+  <xacro:include filename="$(find moveit_resources_pr2_description)/urdf/sensors/wge100_camera.urdf.xacro" />
   <!-- Texture projector -->
-  <xacro:include filename="$(find pr2_description)/urdf/sensors/projector_wg6802418.urdf.xacro" />
+  <xacro:include filename="$(find moveit_resources_pr2_description)/urdf/sensors/projector_wg6802418.urdf.xacro" />
   <!-- generic simulator_gazebo plugins for starting mechanism control, ros time, ros battery -->
-  <xacro:include filename="$(find pr2_description)/gazebo/gazebo.urdf.xacro" />
+  <xacro:include filename="$(find moveit_resources_pr2_description)/gazebo/gazebo.urdf.xacro" />
   <!-- materials for visualization -->
-  <xacro:include filename="$(find pr2_description)/urdf/materials.urdf.xacro" />
+  <xacro:include filename="$(find moveit_resources_pr2_description)/urdf/materials.urdf.xacro" />
   <!-- Now we can start using the macros included above to define the actual PR2 -->
   <!-- The first use of a macro.  This one was defined in base.urdf.xacro above.

File: pr2_description/robots/pr2_se.urdf.xacro (robot description, xacro)
@@ -3,30 +3,30 @@
   <!-- The following included files set up definitions of parts of the robot body -->
   <!-- misc common stuff? -->
-  <xacro:include filename="$(find pr2_description)/urdf/common.xacro" />
+  <xacro:include filename="$(find moveit_resources_pr2_description)/urdf/common.xacro" />
   <!-- PR2 Arm -->
-  <xacro:include filename="$(find pr2_description)/urdf/shoulder_v0/shoulder.urdf.xacro" />
-  <xacro:include filename="$(find pr2_description)/urdf/upper_arm_v0/upper_arm.urdf.xacro" />
-  <xacro:include filename="$(find pr2_description)/urdf/forearm_v0/forearm.urdf.xacro" />
+  <xacro:include filename="$(find moveit_resources_pr2_description)/urdf/shoulder_v0/shoulder.urdf.xacro" />
+  <xacro:include filename="$(find moveit_resources_pr2_description)/urdf/upper_arm_v0/upper_arm.urdf.xacro" />
+  <xacro:include filename="$(find moveit_resources_pr2_description)/urdf/forearm_v0/forearm.urdf.xacro" />
   <!-- PR2 gripper -->
-  <xacro:include filename="$(find pr2_description)/urdf/gripper_v0/gripper.urdf.xacro" />
+  <xacro:include filename="$(find moveit_resources_pr2_description)/urdf/gripper_v0/gripper.urdf.xacro" />
   <!-- PR2 head -->
-  <xacro:include filename="$(find pr2_description)/urdf/head_v0/head.urdf.xacro" />
+  <xacro:include filename="$(find moveit_resources_pr2_description)/urdf/head_v0/head.urdf.xacro" />
   <!-- PR2 tilting laser mount -->
-  <xacro:include filename="$(find pr2_description)/urdf/tilting_laser_v0/tilting_laser.urdf.xacro" />
+  <xacro:include filename="$(find moveit_resources_pr2_description)/urdf/tilting_laser_v0/tilting_laser.urdf.xacro" />
   <!-- PR2 torso -->
-  <xacro:include filename="$(find pr2_description)/urdf/torso_v0/torso.urdf.xacro" />
+  <xacro:include filename="$(find moveit_resources_pr2_description)/urdf/torso_v0/torso.urdf.xacro" />
   <!-- PR2 base -->
-  <xacro:include filename="$(find pr2_description)/urdf/base_v0/base.urdf.xacro" />
+  <xacro:include filename="$(find moveit_resources_pr2_description)/urdf/base_v0/base.urdf.xacro" />
   <!-- Head sensors -->
   <!-- kinect/prosilica model -->
-  <xacro:include filename="$(find pr2_description)/urdf/sensors/kinect_prosilica_camera.urdf.xacro" />
+  <xacro:include filename="$(find moveit_resources_pr2_description)/urdf/sensors/kinect_prosilica_camera.urdf.xacro" />
   <!-- Camera sensors -->
-  <xacro:include filename="$(find pr2_description)/urdf/sensors/wge100_camera.urdf.xacro" />
+  <xacro:include filename="$(find moveit_resources_pr2_description)/urdf/sensors/wge100_camera.urdf.xacro" />
   <!-- Texture projector -->
-  <xacro:include filename="$(find pr2_description)/urdf/sensors/projector_wg6802418.urdf.xacro" />
+  <xacro:include filename="$(find moveit_resources_pr2_description)/urdf/sensors/projector_wg6802418.urdf.xacro" />
   <!-- generic simulator_gazebo plugins for starting mechanism control, ros time, ros battery -->
-  <xacro:include filename="$(find pr2_description)/gazebo/gazebo.urdf.xacro" />
+  <xacro:include filename="$(find moveit_resources_pr2_description)/gazebo/gazebo.urdf.xacro" />
   <!-- materials for visualization -->
-  <xacro:include filename="$(find pr2_description)/urdf/materials.urdf.xacro" />
+  <xacro:include filename="$(find moveit_resources_pr2_description)/urdf/materials.urdf.xacro" />
   <!-- Now we can start using the macros included above to define the actual PR2 -->
   <!-- The first use of a macro.  This one was defined in base.urdf.xacro above.

File: pr2_description/urdf/base_v0/base.urdf.xacro (robot description, xacro)
@@ -1,7 +1,7 @@
 <?xml version="1.0"?>
 <robot xmlns:xacro="http://www.ros.org/wiki/xacro">
-  <xacro:include filename="$(find pr2_description)/urdf/sensors/hokuyo_lx30_laser.urdf.xacro" />
-  <xacro:include filename="$(find pr2_description)/urdf/base_v0/base.gazebo.xacro" />
-  <xacro:include filename="$(find pr2_description)/urdf/base_v0/base.transmission.xacro" />
+  <xacro:include filename="$(find moveit_resources_pr2_description)/urdf/sensors/hokuyo_lx30_laser.urdf.xacro" />
+  <xacro:include filename="$(find moveit_resources_pr2_description)/urdf/base_v0/base.gazebo.xacro" />
+  <xacro:include filename="$(find moveit_resources_pr2_description)/urdf/base_v0/base.transmission.xacro" />
   <!-- DATA SOURCES -->
   <!-- all link offsets, CG, limits are obtained from Function Engineering spreadsheet 090224_link_data.xls unless stated otherwise -->
@@ -55,5 +55,5 @@
         <origin xyz="0 0 0" rpy="0 0 0" />
         <geometry>
-          <mesh filename="package://pr2_description/meshes/base_v0/wheel.dae" />
+          <mesh filename="package://moveit_resources_pr2_description/meshes/base_v0/wheel.dae" />
         </geometry>
         <material name="Wheel_${suffix}" />
@@ -92,5 +92,5 @@
         <origin xyz="0 0 0" rpy="0 0 0" />
         <geometry>
-          <mesh filename="package://pr2_description/meshes/base_v0/caster.stl" />
+          <mesh filename="package://moveit_resources_pr2_description/meshes/base_v0/caster.stl" />
         </geometry>
         <material name="Caster" />
@@ -99,5 +99,5 @@
         <origin xyz="0 0 0" rpy="0 0 0" />
         <geometry>
-          <mesh filename="package://pr2_description/meshes/base_v0/caster_L.stl" />
+          <mesh filename="package://moveit_resources_pr2_description/meshes/base_v0/caster_L.stl" />
         </geometry>
       </collision>
@@ -129,5 +129,5 @@
         <origin xyz="0 0 0" rpy="0 0 0" />
         <geometry>
-          <mesh filename="package://pr2_description/meshes/base_v0/base.dae" />
+          <mesh filename="package://moveit_resources_pr2_description/meshes/base_v0/base.dae" />
         </geometry>
         <material name="White" />
@@ -136,5 +136,5 @@
         <origin xyz="0 0 0" rpy="0 0 0" />
         <geometry>
-          <mesh filename="package://pr2_description/meshes/base_v0/base_L.stl" />
+          <mesh filename="package://moveit_resources_pr2_description/meshes/base_v0/base_L.stl" />
         </geometry>
       </collision>

File: pr2_description/urdf/forearm_v0/forearm.urdf.xacro (robot description, xacro)
@@ -4,7 +4,7 @@
   <!-- Things that are needed only for Gazebo (not the physical robot).  These include
        sensor and controller plugin specifications -->
-  <xacro:include filename="$(find pr2_description)/urdf/forearm_v0/forearm.gazebo.xacro" />
-  <xacro:include filename="$(find pr2_description)/urdf/forearm_v0/forearm.transmission.xacro" />
-  <xacro:include filename="$(find pr2_description)/urdf/common.xacro" />
+  <xacro:include filename="$(find moveit_resources_pr2_description)/urdf/forearm_v0/forearm.gazebo.xacro" />
+  <xacro:include filename="$(find moveit_resources_pr2_description)/urdf/forearm_v0/forearm.transmission.xacro" />
+  <xacro:include filename="$(find moveit_resources_pr2_description)/urdf/common.xacro" />
   <!-- ============================   Forearm   ============================ -->
   <xacro:macro name="pr2_forearm_v0" params="side parent reflect *origin
@@ -27,5 +27,5 @@
         <origin xyz="0 0 0" rpy="0 0 0" />
         <geometry>
-          <mesh filename="package://pr2_description/meshes/forearm_v0/forearm.dae" />
+          <mesh filename="package://moveit_resources_pr2_description/meshes/forearm_v0/forearm.dae" />
        </geometry>
         <material name="Grey" />
@@ -34,5 +34,5 @@
         <origin xyz="0 0 0" rpy="0 0 0" />
         <geometry>
-          <mesh filename="package://pr2_description/meshes/forearm_v0/forearm.stl" />
+          <mesh filename="package://moveit_resources_pr2_description/meshes/forearm_v0/forearm.stl" />
         </geometry>
       </collision>
@@ -65,5 +65,5 @@
         <origin xyz="0 0 0" rpy="0 0 0" />
         <geometry>
-          <mesh filename="package://pr2_description/meshes/forearm_v0/wrist_flex.dae" />
+          <mesh filename="package://moveit_resources_pr2_description/meshes/forearm_v0/wrist_flex.dae" />
         </geometry>
         <material name="Grey" />
@@ -72,5 +72,5 @@
         <origin xyz="0 0 0" rpy="0 0 0" />
         <geometry>
-          <mesh filename="package://pr2_description/meshes/forearm_v0/wrist_flex.stl" />
+          <mesh filename="package://moveit_resources_pr2_description/meshes/forearm_v0/wrist_flex.stl" />
         </geometry>
       </collision>
@@ -104,5 +104,5 @@
         <origin xyz="0 0 0" rpy="0 0 0" />
         <geometry>
-          <mesh filename="package://pr2_description/meshes/forearm_v0/wrist_roll.stl" />
+          <mesh filename="package://moveit_resources_pr2_description/meshes/forearm_v0/wrist_roll.stl" />
         </geometry>
         <material name="RollLinks" />
@@ -111,5 +111,5 @@
         <origin xyz="0 0 0" rpy="0 0 0" />
         <geometry>
-          <mesh filename="package://pr2_description/meshes/forearm_v0/wrist_roll_L.stl" />
+          <mesh filename="package://moveit_resources_pr2_description/meshes/forearm_v0/wrist_roll_L.stl" />
         </geometry>
       </collision>
