Commit message: Add moveit_resources_ prefix to pr2_description

File: pr2_description/urdf/gripper_v0/gripper.urdf.xacro (robot description, xacro)
@@ -1,6 +1,6 @@
 <?xml version="1.0"?>
 <robot xmlns:xacro="http://www.ros.org/wiki/xacro">
-  <xacro:include filename="$(find pr2_description)/urdf/gripper_v0/gripper.gazebo.xacro" />
-  <xacro:include filename="$(find pr2_description)/urdf/gripper_v0/gripper.transmission.xacro" />
+  <xacro:include filename="$(find moveit_resources_pr2_description)/urdf/gripper_v0/gripper.gazebo.xacro" />
+  <xacro:include filename="$(find moveit_resources_pr2_description)/urdf/gripper_v0/gripper.transmission.xacro" />
   <xacro:property name="M_PI" value="3.1415926535897931" />
   <xacro:property name="gripper_upper_angle" value="0.548" />
@@ -45,5 +45,5 @@
         <origin xyz="0 0 0" rpy="0 0 0" />
         <geometry>
-          <mesh filename="package://pr2_description/meshes/gripper_v0/l_finger.dae" />
+          <mesh filename="package://moveit_resources_pr2_description/meshes/gripper_v0/l_finger.dae" />
         </geometry>
         <material name="Grey" />
@@ -52,5 +52,5 @@
         <origin xyz="0 0 0" rpy="0 0 0" />
         <geometry>
-          <mesh filename="package://pr2_description/meshes/gripper_v0/l_finger.stl" />
+          <mesh filename="package://moveit_resources_pr2_description/meshes/gripper_v0/l_finger.stl" />
         </geometry>
       </collision>
@@ -80,5 +80,5 @@
         <origin xyz="0 0 0" rpy="${M_PI} 0 0" />
         <geometry>
-          <mesh filename="package://pr2_description/meshes/gripper_v0/l_finger.dae" />
+          <mesh filename="package://moveit_resources_pr2_description/meshes/gripper_v0/l_finger.dae" />
         </geometry>
         <material name="Grey" />
@@ -87,5 +87,5 @@
         <origin xyz="0 0 0" rpy="${M_PI} 0 0" />
         <geometry>
-          <mesh filename="package://pr2_description/meshes/gripper_v0/l_finger.stl" />
+          <mesh filename="package://moveit_resources_pr2_description/meshes/gripper_v0/l_finger.stl" />
         </geometry>
       </collision>
@@ -112,5 +112,5 @@
         <origin xyz="0 0 0" rpy="0 0 0" />
         <geometry>
-          <mesh filename="package://pr2_description/meshes/gripper_v0/l_finger_tip.dae" />
+          <mesh filename="package://moveit_resources_pr2_description/meshes/gripper_v0/l_finger_tip.dae" />
         </geometry>
         <material name="Green" />
@@ -119,5 +119,5 @@
         <origin xyz="0 0 0" rpy="0 0 0" />
         <geometry>
-          <mesh filename="package://pr2_description/meshes/gripper_v0/l_finger_tip.stl" />
+          <mesh filename="package://moveit_resources_pr2_description/meshes/gripper_v0/l_finger_tip.stl" />
         </geometry>
       </collision>
@@ -144,5 +144,5 @@
         <origin xyz="0 0 0" rpy="${M_PI} 0 0" />
         <geometry>
-          <mesh filename="package://pr2_description/meshes/gripper_v0/l_finger_tip.dae"  />
+          <mesh filename="package://moveit_resources_pr2_description/meshes/gripper_v0/l_finger_tip.dae"  />
         </geometry>
         <material name="Green" />
@@ -151,5 +151,5 @@
         <origin xyz="0 0 0" rpy="${M_PI} 0 0" />
         <geometry>
-          <mesh filename="package://pr2_description/meshes/gripper_v0/l_finger_tip.stl"  />
+          <mesh filename="package://moveit_resources_pr2_description/meshes/gripper_v0/l_finger_tip.stl"  />
         </geometry>
       </collision>
@@ -175,5 +175,5 @@
         <origin xyz="0 0 0" rpy="0 0 0" />
         <geometry>
-          <mesh filename="package://pr2_description/meshes/gripper_v0/gripper_palm.dae"  />
+          <mesh filename="package://moveit_resources_pr2_description/meshes/gripper_v0/gripper_palm.dae"  />
         </geometry>
         <material name="Red" />
@@ -182,5 +182,5 @@
         <origin xyz="0 0 0" rpy="0 0 0" />
         <geometry>
-          <mesh filename="package://pr2_description/meshes/gripper_v0/gripper_palm.stl"  />
+          <mesh filename="package://moveit_resources_pr2_description/meshes/gripper_v0/gripper_palm.stl"  />
         </geometry>
       </collision>

File: pr2_description/urdf/head_v0/head.urdf.xacro (robot description, xacro)
@@ -1,6 +1,6 @@
 <?xml version="1.0"?>
 <robot xmlns:xacro="http://www.ros.org/wiki/xacro">
-  <xacro:include filename="$(find pr2_description)/urdf/head_v0/head.gazebo.xacro" />
-  <xacro:include filename="$(find pr2_description)/urdf/head_v0/head.transmission.xacro" />
+  <xacro:include filename="$(find moveit_resources_pr2_description)/urdf/head_v0/head.gazebo.xacro" />
+  <xacro:include filename="$(find moveit_resources_pr2_description)/urdf/head_v0/head.transmission.xacro" />
   <xacro:property name="M_PI" value="3.1415926535897931" />
   <xacro:macro name="pr2_head_pan_v0" params="name parent *origin head_pan_calib_ref:=0.0">
@@ -25,5 +25,5 @@
         <origin xyz="0 0 0.0" rpy="0 0 0 " />
         <geometry>
-          <mesh filename="package://pr2_description/meshes/head_v0/head_pan.dae"  />
+          <mesh filename="package://moveit_resources_pr2_description/meshes/head_v0/head_pan.dae"  />
         </geometry>
         <material name="Blue" />
@@ -31,5 +31,5 @@
       <collision>
         <geometry>
-          <mesh filename="package://pr2_description/meshes/head_v0/head_pan_L.stl"  />
+          <mesh filename="package://moveit_resources_pr2_description/meshes/head_v0/head_pan_L.stl"  />
         </geometry>
       </collision>
@@ -65,5 +65,5 @@
         <origin xyz="0 0 0" rpy="0.0 0.0 0.0" />
         <geometry>
-          <mesh filename="package://pr2_description/meshes/head_v0/head_tilt.dae"  />
+          <mesh filename="package://moveit_resources_pr2_description/meshes/head_v0/head_tilt.dae"  />
         </geometry>
         <material name="Green" />
@@ -72,5 +72,5 @@
         <origin xyz="0 0 0" rpy="0.0 0.0 0.0" />
         <geometry>
-          <mesh filename="package://pr2_description/meshes/head_v0/head_tilt_L.stl"  />
+          <mesh filename="package://moveit_resources_pr2_description/meshes/head_v0/head_tilt_L.stl"  />
         </geometry>
       </collision>

File: pr2_description/urdf/sensors/double_stereo_camera.urdf.xacro (robot description, xacro)
@@ -1,6 +1,6 @@
 <?xml version="1.0"?>
 <robot xmlns:xacro="http://www.ros.org/wiki/xacro">
-  <xacro:include filename="$(find pr2_description)/urdf/sensors/double_stereo_camera.gazebo.xacro" />
-  <xacro:include filename="$(find pr2_description)/urdf/sensors/stereo_camera.urdf.xacro" />
+  <xacro:include filename="$(find moveit_resources_pr2_description)/urdf/sensors/double_stereo_camera.gazebo.xacro" />
+  <xacro:include filename="$(find moveit_resources_pr2_description)/urdf/sensors/stereo_camera.urdf.xacro" />
   <xacro:property name="stereo_size_x" value="0.02" />
   <xacro:property name="stereo_size_y" value="0.12" />

File: pr2_description/urdf/sensors/head_sensor_package.urdf.xacro (robot description, xacro)
@@ -5,7 +5,7 @@
        double stereo camera
   -->
-  <xacro:include filename="$(find pr2_description)/urdf/sensors/head_sensor_package.gazebo.xacro" />
-  <xacro:include filename="$(find pr2_description)/urdf/sensors/double_stereo_camera.urdf.xacro" />
-  <xacro:include filename="$(find pr2_description)/urdf/sensors/prosilica_gc2450_camera.urdf.xacro" />
+  <xacro:include filename="$(find moveit_resources_pr2_description)/urdf/sensors/head_sensor_package.gazebo.xacro" />
+  <xacro:include filename="$(find moveit_resources_pr2_description)/urdf/sensors/double_stereo_camera.urdf.xacro" />
+  <xacro:include filename="$(find moveit_resources_pr2_description)/urdf/sensors/prosilica_gc2450_camera.urdf.xacro" />
   <!-- Made by Kevin for A2 sensor package -->
   <!-- Origin is center mount screw on sensor plate mount -->

File: pr2_description/urdf/sensors/hokuyo_lx30_laser.urdf.xacro (robot description, xacro)
@@ -1,5 +1,5 @@
 <?xml version="1.0"?>
 <robot xmlns:xacro="http://www.ros.org/wiki/xacro">
-  <xacro:include filename="$(find pr2_description)/urdf/sensors/hokuyo_lx30_laser.gazebo.xacro" />
+  <xacro:include filename="$(find moveit_resources_pr2_description)/urdf/sensors/hokuyo_lx30_laser.gazebo.xacro" />
   <xacro:macro name="hokuyo_lx30_laser_v0" params="name parent *origin ros_topic update_rate min_angle max_angle">
     <joint name="${name}_joint" type="fixed">

File: pr2_description/urdf/sensors/kinect2.urdf.xacro (robot description, xacro)
@@ -1,5 +1,5 @@
 <?xml version="1.0"?>
 <robot xmlns:xacro="http://www.ros.org/wiki/xacro">
-  <xacro:include filename="$(find pr2_description)/urdf/sensors/kinect2.gazebo.xacro" />
+  <xacro:include filename="$(find moveit_resources_pr2_description)/urdf/sensors/kinect2.gazebo.xacro" />
   <xacro:property name="ir_depth_rgb_offset_y" value="0.01"/> <!-- FIXME: what is this offset? -->
   <!-- Kinect2 and mount assembly -->
@@ -21,5 +21,5 @@
         <origin xyz="-0.102 -0.148 0" rpy="0 0 0"/>
         <geometry>
-          <mesh filename="package://pr2_description/meshes/sensors/kinect2_v0/kinect2_assembly.dae" scale="0.001 0.001 0.001" />
+          <mesh filename="package://moveit_resources_pr2_description/meshes/sensors/kinect2_v0/kinect2_assembly.dae" scale="0.001 0.001 0.001" />
         </geometry>
         <material name="gray">

File: pr2_description/urdf/sensors/kinect_camera.urdf.xacro (robot description, xacro)
@@ -1,5 +1,5 @@
 <?xml version="1.0"?>
 <robot xmlns:xacro="http://www.ros.org/wiki/xacro">
-  <xacro:include filename="$(find pr2_description)/urdf/sensors/kinect_camera.gazebo.xacro" />
+  <xacro:include filename="$(find moveit_resources_pr2_description)/urdf/sensors/kinect_camera.gazebo.xacro" />
   <xacro:macro name="kinect_camera_v0" params="name parent *origin">
     <joint name="${name}_frame_joint" type="fixed">
@@ -19,5 +19,5 @@
         <origin xyz="0.0 0.012 0" rpy="0 0 0"/>
         <geometry>
-          <mesh filename="package://pr2_description/meshes/sensors/kinect_v0/kinect.dae" scale="0.001 0.001 0.001" />
+          <mesh filename="package://moveit_resources_pr2_description/meshes/sensors/kinect_v0/kinect.dae" scale="0.001 0.001 0.001" />
         </geometry>
       </visual>
@@ -25,5 +25,5 @@
         <origin xyz="0.0 0.012 0" rpy="0 0 0"/>
         <geometry>
-          <mesh filename="package://pr2_description/meshes/sensors/kinect_v0/kinect.dae" scale="0.001 0.001 0.001" />
+          <mesh filename="package://moveit_resources_pr2_description/meshes/sensors/kinect_v0/kinect.dae" scale="0.001 0.001 0.001" />
         </geometry>
       </collision>

File: pr2_description/urdf/sensors/kinect_prosilica_camera.urdf.xacro (robot description, xacro)
@@ -1,5 +1,5 @@
 <?xml version="1.0"?>
 <root xmlns:xacro="http://www.ros.org/wiki/xacro">
-  <xacro:include filename="$(find pr2_description)/urdf/sensors/kinect_prosilica_camera.gazebo.xacro" />
+  <xacro:include filename="$(find moveit_resources_pr2_description)/urdf/sensors/kinect_prosilica_camera.gazebo.xacro" />
   <xacro:property name="ir_depth_rgb_offset_y" value="0.01"/> <!-- FIXME: what is this offset? -->
   <!-- kinect and prosilica combo -->
@@ -24,5 +24,5 @@
         <origin xyz="0.0 0.0 0" rpy="0 0 0"/>
         <geometry>
-          <mesh filename="package://pr2_description/meshes/sensors/kinect_prosilica_v0/115x100_swept_back--coarse.STL" scale="0.001 0.001 0.001" />
+          <mesh filename="package://moveit_resources_pr2_description/meshes/sensors/kinect_prosilica_v0/115x100_swept_back--coarse.STL" scale="0.001 0.001 0.001" />
         </geometry>
         <material name="gray">

File: pr2_description/urdf/sensors/microstrain_3dmgx2_imu.urdf.xacro (robot description, xacro)
@@ -1,5 +1,5 @@
 <?xml version="1.0"?>
 <robot xmlns:xacro="http://www.ros.org/wiki/xacro">
-  <xacro:include filename="$(find pr2_description)/urdf/sensors/microstrain_3dmgx2_imu.gazebo.xacro" />
+  <xacro:include filename="$(find moveit_resources_pr2_description)/urdf/sensors/microstrain_3dmgx2_imu.gazebo.xacro" />
   <xacro:macro name="microstrain_3dmgx2_imu_v0" params="name parent *origin imu_topic update_rate stdev">
     <joint name="${name}_joint" type="fixed">

File: pr2_description/urdf/sensors/projector_wg6802418.urdf.xacro (robot description, xacro)
@@ -1,5 +1,5 @@
 <?xml version="1.0"?>
 <root xmlns:xacro="http://www.ros.org/wiki/xacro">
-  <xacro:include filename="$(find pr2_description)/urdf/sensors/projector_wg6802418.gazebo.xacro" />
+  <xacro:include filename="$(find moveit_resources_pr2_description)/urdf/sensors/projector_wg6802418.gazebo.xacro" />
   <xacro:macro name="projector_wg6802418_v0" params="name parent *origin">
     <joint name="${name}_frame_joint" type="fixed">

File: pr2_description/urdf/sensors/prosilica_gc2450_camera.urdf.xacro (robot description, xacro)
@@ -1,5 +1,5 @@
 <?xml version="1.0"?>
 <root xmlns:xacro="http://www.ros.org/wiki/xacro">
-  <xacro:include filename="$(find pr2_description)/urdf/sensors/prosilica_gc2450_camera.gazebo.xacro" />
+  <xacro:include filename="$(find moveit_resources_pr2_description)/urdf/sensors/prosilica_gc2450_camera.gazebo.xacro" />
   <xacro:macro name="prosilica_cam_v0" params="frame_name parent *origin camera_name">
     <joint name="${frame_name}_frame_joint" type="fixed">

File: pr2_description/urdf/sensors/stereo_camera.urdf.xacro (robot description, xacro)
@@ -2,6 +2,6 @@
 <robot xmlns:xacro="http://www.ros.org/wiki/xacro">
   <!-- stereo camera macro uses wge100_camera macros -->
-  <xacro:include filename="$(find pr2_description)/urdf/sensors/wge100_camera.urdf.xacro" />
-  <xacro:include filename="$(find pr2_description)/urdf/sensors/stereo_camera.gazebo.xacro" />
+  <xacro:include filename="$(find moveit_resources_pr2_description)/urdf/sensors/wge100_camera.urdf.xacro" />
+  <xacro:include filename="$(find moveit_resources_pr2_description)/urdf/sensors/stereo_camera.gazebo.xacro" />
   <xacro:property name="stereo_dx" value="0.00" />
   <xacro:property name="stereo_dy" value="-0.09" /> <!-- +y to the left -->

File: pr2_description/urdf/sensors/wge100_camera.urdf.xacro (robot description, xacro)
@@ -2,5 +2,5 @@
 <!-- XML namespaces -->
 <robot xmlns:xacro="http://www.ros.org/wiki/xacro">
-  <xacro:include filename="$(find pr2_description)/urdf/sensors/wge100_camera.gazebo.xacro" />
+  <xacro:include filename="$(find moveit_resources_pr2_description)/urdf/sensors/wge100_camera.gazebo.xacro" />
   <!-- hack_baseline is used to simulate right stereo camera projection matrix translation to left stereo camera frame, currently on the hardware,
        custom left stereo camera frame_id is passed to right stereo wge100 camera node at launch time, baseline is stored on the camera. -->

File: pr2_description/urdf/shoulder_v0/shoulder.urdf.xacro (robot description, xacro)
@@ -4,7 +4,7 @@
   <!-- Things that are needed only for Gazebo (not the physical robot).  These include
        sensor and controller plugin specifications -->
-  <xacro:include filename="$(find pr2_description)/urdf/shoulder_v0/shoulder.gazebo.xacro" />
-  <xacro:include filename="$(find pr2_description)/urdf/shoulder_v0/shoulder.transmission.xacro" />
-  <xacro:include filename="$(find pr2_description)/urdf/common.xacro" />
+  <xacro:include filename="$(find moveit_resources_pr2_description)/urdf/shoulder_v0/shoulder.gazebo.xacro" />
+  <xacro:include filename="$(find moveit_resources_pr2_description)/urdf/shoulder_v0/shoulder.transmission.xacro" />
+  <xacro:include filename="$(find moveit_resources_pr2_description)/urdf/common.xacro" />
   <xacro:property name="shoulder_lift_length" value="0.10" />  <!--TODO Define and give source-->
   <xacro:property name="shoulder_lift_radius" value="0.12" />  <!--TODO Define and give source-->
@@ -45,5 +45,5 @@
         <origin xyz="0 0 0" rpy="0 0 0" />
         <geometry>
-          <mesh filename="package://pr2_description/meshes/shoulder_v0/shoulder_pan.dae"  />
+          <mesh filename="package://moveit_resources_pr2_description/meshes/shoulder_v0/shoulder_pan.dae"  />
         </geometry>
         <material name="Blue" />
@@ -52,5 +52,5 @@
         <origin xyz="0.0 0 0.0" rpy="0 0 0" />
         <geometry>
-          <mesh filename="package://pr2_description/meshes/shoulder_v0/shoulder_pan.stl"  />
+          <mesh filename="package://moveit_resources_pr2_description/meshes/shoulder_v0/shoulder_pan.stl"  />
         </geometry>
       </collision>
@@ -86,5 +86,5 @@
         <origin xyz="0 0 0" rpy="0 0 0" />
         <geometry>
-          <mesh filename="package://pr2_description/meshes/shoulder_v0/shoulder_lift.dae"  />
+          <mesh filename="package://moveit_resources_pr2_description/meshes/shoulder_v0/shoulder_lift.dae"  />
         </geometry>
         <material name="Grey" />
@@ -93,5 +93,5 @@
         <origin xyz="0 0 0" rpy="0 0 0" />
         <geometry>
-          <mesh filename="package://pr2_description/meshes/shoulder_v0/shoulder_lift.stl"  />
+          <mesh filename="package://moveit_resources_pr2_description/meshes/shoulder_v0/shoulder_lift.stl"  />
         </geometry>
       </collision>
@@ -137,5 +137,5 @@
         <origin xyz="0 0 0" rpy="0 0 0" />
         <geometry>
-          <mesh filename="package://pr2_description/meshes/shoulder_v0/upper_arm_roll.stl"  />
+          <mesh filename="package://moveit_resources_pr2_description/meshes/shoulder_v0/upper_arm_roll.stl"  />
         </geometry>
         <material name="RollLinks" />
@@ -144,5 +144,5 @@
         <origin xyz="0 0 0" rpy="0 0 0" />
         <geometry>
-          <mesh filename="package://pr2_description/meshes/shoulder_v0/upper_arm_roll_L.stl"  />
+          <mesh filename="package://moveit_resources_pr2_description/meshes/shoulder_v0/upper_arm_roll_L.stl"  />
         </geometry>
       </collision>
